File: outputs/PCIe_AllM2_RevP/Main_20M2/Main_20M2.kicad_pcb (KiCad board)
At the start: 32 copper layers, 120 x 45 mm, 643 parts, among them J11 12V 25A FEED / DESIGN TARGET,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, J12 12V 25A FEED / DESIGN TARGET,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, J401 CUSTOM 12V POWER / SMT SHELL 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, J402 TB5 PORT / SMT SHELL DRAFT / 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, J501 M1 SSD / VERTICAL M-Key 2280 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, J502 M2 SSD / VERTICAL M-Key 2280 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, J503 M3 SSD / VERTICAL M-Key 2280 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, J504 M4 SSD / VERTICAL M-Key 2280 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, J6001 N01 M-Key 2280 / x4 / NO-PEG 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, J6002 N02 M-Key 2280 / x4 / NO-PEG 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, J6003 N03 M-Key 2280 / x4 / NO-PEG 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, J6004 N04 M-Key 2280 / x4 / NO-PEG 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, J6005 N05 M-Key 2280 / x4 / NO-PEG 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, J6006 N06 M-Key 2280 / x4 / NO-PEG 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, J6007 N07 M-Key 2280 / x4 / NO-PEG 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, J6008 N08 M-Key 2280 / x4 / NO-PEG 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, J6009 N09 M-Key 2280 / x4 / NO-PEG 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, J6010 N10 M-Key 2280 / x4 / NO-PEG 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, J6011 N11 M-Key 2280 / x4 / NO-PEG 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, J6012 N12 M-Key 2280 / x4 / NO-PEG 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, J6013 N13 M-Key 2280 / x4 / NO-PEG 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, J6014 N14 M-Key 2280 / x4 / NO-PEG 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, J6015 N15 M-Key 2280 / x4 / NO-PEG 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, J6016 N16 M-Key 2280 / x4 / NO-PEG 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, U1 Broadcom PEX88096 / SS02-0B00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, U30 TPS259470ARPWR, U3001 TPS565201DDCR, U3002 TPS565201DDCR, U3003 TPS565201DDCR, U3004 TPS565201DDCR, U31 TPS62132RGTR, U41 TPS259470ARPWR, U42 TPS259470ARPWR, U5001 TPSM53604RDAR / 12V to 3.3V 4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, U5002 TPSM53604RDAR / 12V to 3.3V 4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, U5003 TPSM53604RDAR / 12V to 3.3V 4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, U5004 TPSM53604RDAR / 12V to 3.3V 4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, U5005 TPSM53604RDAR / 12V to 3.3V 4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, U5006 TPSM53604RDAR / 12V to 3.3V 4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, U5007 TPSM53604RDAR / 12V to 3.3V 4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, U5008 TPSM53604RDAR / 12V to 3.3V 4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, U5009 TPSM53604RDAR / 12V to 3.3V 4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, U501 Intel_JHL9580_MECH_13x13_UNVE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, U5010 TPSM53604RDAR / 12V to 3.3V 4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, U5011 TPSM53604RDAR / 12V to 3.3V 4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, U5012 TPSM53604RDAR / 12V to 3.3V 4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, U5013 TPSM53604RDAR / 12V to 3.3V 4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, U5014 TPSM53604RDAR / 12V to 3.3V 4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, U5015 TPSM53604RDAR / 12V to 3.3V 4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, U5016 TPSM53604RDAR / 12V to 3.3V 4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, U502 Intel Core Ultra 7 268V / BGA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, U601 9ZXL0851EKILFT / CPU common c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, U602 9ZXL0851EKILFT / CPU common c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, U603 9FGV0241AKLF / DNP ALTERNATE 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, U604 9DML0451AKILF / DNP ALTERNATE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, U605 TPS3808G09DBVR / SUPPORT NETW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, U606 W25Q32JWSSIQ_C2980995 / SUPPO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, U607 TCA9548ARGER / SUPPORT NETWOR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, U6501 9ZXL0851EKILFT / N12-N16 CLOC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, U701 W25Q256JWPIQ / 1.8V 32MiB BIOS, U702 TPS7A0215PDBVR / RTC 1.5V, Y701 38.4MHz crystal / load and ES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, Y702 32.768kHz crystal / load and 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

Commit message: Repair Rev P reset bias, native parity and netclass validation
Parts:
- added R3005: 100k / RESET BIAS ONLY - RELEASE DRIVER PENDING, Local:R_0402_1005Metric, F.Cu at (6.00, 28.0)
- added R3015: 100k / RESET BIAS ONLY - RELEASE DRIVER PENDING, Local:R_0402_1005Metric, F.Cu at (12.0, 28.0)
- added R3025: 100k / RESET BIAS ONLY - RELEASE DRIVER PENDING, Local:R_0402_1005Metric, F.Cu at (108.0, 28.0)
- added R3035: 100k / RESET BIAS ONLY - RELEASE DRIVER PENDING, Local:R_0402_1005Metric, F.Cu at (114.0, 28.0)
Connections:
- net /AUX_12V_PROTECTED renamed /AUX_12V_PROTECTED
- net /AUX_DVDT renamed /AUX_DVDT
- net /AUX_ILM renamed /AUX_ILM
- net /AUX_OV renamed /AUX_OV
- net /AUX_PG renamed /AUX_PG
- net /AUX_UV renamed /AUX_UV
- net /BUCK_SS renamed /BUCK_SS
- net /BUCK_SW renamed /BUCK_SW
- net /CLKBUF1_VDDA renamed /CLKBUF1_VDDA
- net /CLKBUF2_VDDA renamed /CLKBUF2_VDDA
- net /CLKBUF3_VDDA renamed /CLKBUF3_VDDA
- net /CPU_ACPRESENT renamed /CPU_ACPRESENT
- net /CPU_BATLOW_N renamed /CPU_BATLOW_N
- net /CPU_CLKBUF1_IN_N renamed /CPU_CLKBUF1_IN_N
- net /CPU_CLKBUF1_IN_P renamed /CPU_CLKBUF1_IN_P
- net /CPU_CLKBUF2_IN_N renamed /CPU_CLKBUF2_IN_N
- net /CPU_CLKBUF2_IN_P renamed /CPU_CLKBUF2_IN_P
- net /CPU_CLKBUF3_IN_N renamed /CPU_CLKBUF3_IN_N
- net /CPU_CLKBUF3_IN_P renamed /CPU_CLKBUF3_IN_P
- net /CPU_CLKREQ0_N renamed /CPU_CLKREQ0_N
- net /CPU_CLKREQ1_N renamed /CPU_CLKREQ1_N
- net /CPU_CLKREQ2_N renamed /CPU_CLKREQ2_N
- net /CPU_CLK_RCOMP renamed /CPU_CLK_RCOMP
- net /CPU_EPD_ON_LOOP_1V25 renamed /CPU_EPD_ON_LOOP_1V25
- net /CPU_G5_RX0_N renamed /CPU_G5_RX0_N
- net /CPU_G5_RX0_P renamed /CPU_G5_RX0_P
- net /CPU_G5_RX1_N renamed /CPU_G5_RX1_N
- net /CPU_G5_RX1_P renamed /CPU_G5_RX1_P
- net /CPU_G5_RX2_N renamed /CPU_G5_RX2_N
- net /CPU_G5_RX2_P renamed /CPU_G5_RX2_P
- net /CPU_G5_RX3_N renamed /CPU_G5_RX3_N
- net /CPU_G5_RX3_P renamed /CPU_G5_RX3_P
- net /CPU_G5_TX0_N renamed /CPU_G5_TX0_N
- net /CPU_G5_TX0_P renamed /CPU_G5_TX0_P
- net /CPU_G5_TX1_N renamed /CPU_G5_TX1_N
- net /CPU_G5_TX1_P renamed /CPU_G5_TX1_P
- net /CPU_G5_TX2_N renamed /CPU_G5_TX2_N
- net /CPU_G5_TX2_P renamed /CPU_G5_TX2_P
- net /CPU_G5_TX3_N renamed /CPU_G5_TX3_N
- net /CPU_G5_TX3_P renamed /CPU_G5_TX3_P
- net /CPU_PCIE4_RCOMP renamed /CPU_PCIE4_RCOMP
- net /CPU_PCIE5_RCOMP renamed /CPU_PCIE5_RCOMP
- net /CPU_PERST_1V8_N renamed /CPU_PERST_1V8_N
- net /CPU_PEX_RX0_N renamed /CPU_PEX_RX0_N
- net /CPU_PEX_RX0_P renamed /CPU_PEX_RX0_P
- net /CPU_PEX_RX1_N renamed /CPU_PEX_RX1_N
- net /CPU_PEX_RX1_P renamed /CPU_PEX_RX1_P
- net /CPU_PEX_RX2_N renamed /CPU_PEX_RX2_N
- net /CPU_PEX_RX2_P renamed /CPU_PEX_RX2_P
- net /CPU_PEX_RX3_N renamed /CPU_PEX_RX3_N
- net /CPU_PEX_RX3_P renamed /CPU_PEX_RX3_P
- net /CPU_PEX_TX0_N renamed /CPU_PEX_TX0_N
- net /CPU_PEX_TX0_P renamed /CPU_PEX_TX0_P
- net /CPU_PEX_TX1_N renamed /CPU_PEX_TX1_N
- net /CPU_PEX_TX1_P renamed /CPU_PEX_TX1_P
- net /CPU_PEX_TX2_N renamed /CPU_PEX_TX2_N
- net /CPU_PEX_TX2_P renamed /CPU_PEX_TX2_P
- net /CPU_PEX_TX3_N renamed /CPU_PEX_TX3_N
- net /CPU_PEX_TX3_P renamed /CPU_PEX_TX3_P
- net /CPU_PLT_PWROK renamed /CPU_PLT_PWROK
- net /CPU_PMCALERT_N renamed /CPU_PMCALERT_N
- net /CPU_PWRBTN_1V8_N renamed /CPU_PWRBTN_1V8_N
- net /CPU_REFCLK_N renamed /CPU_REFCLK_N
- net /CPU_REFCLK_P renamed /CPU_REFCLK_P
- net /CPU_RSMRST_N renamed /CPU_RSMRST_N
- net /CPU_RTCRST_N renamed /CPU_RTCRST_N
- net /CPU_RTCX1 renamed /CPU_RTCX1
- net /CPU_RTCX2 renamed /CPU_RTCX2
- net /CPU_SLP_S3_1V8_N renamed /CPU_SLP_S3_1V8_N
- net /CPU_SLP_S4_1V8_N renamed /CPU_SLP_S4_1V8_N
- net /CPU_SLP_S5_1V8_N renamed /CPU_SLP_S5_1V8_N
- net /CPU_SPI_CLK_FLASH renamed /CPU_SPI_CLK_FLASH
- net /CPU_SPI_CLK_PAD renamed /CPU_SPI_CLK_PAD
- net /CPU_SPI_CS0_N renamed /CPU_SPI_CS0_N
- net /CPU_SPI_IO0 renamed /CPU_SPI_IO0
- net /CPU_SPI_IO1 renamed /CPU_SPI_IO1
- net /CPU_SPI_IO2 renamed /CPU_SPI_IO2
- net /CPU_SPI_IO3 renamed /CPU_SPI_IO3
- net /CPU_SRTCRST_N renamed /CPU_SRTCRST_N
- net /CPU_SVID_ALERT_1V25_N renamed /CPU_SVID_ALERT_1V25_N
- net /CPU_SVID_CLK_1V25 renamed /CPU_SVID_CLK_1V25
- net /CPU_SVID_DATA_1V25 renamed /CPU_SVID_DATA_1V25
- net /CPU_SYS_PWROK_1V8 renamed /CPU_SYS_PWROK_1V8
- net /CPU_SYS_RESET_1V8_N renamed /CPU_SYS_RESET_1V8_N
- net /CPU_USB2_RCOMP renamed /CPU_USB2_RCOMP
- net /CPU_USB32_RCOMP renamed /CPU_USB32_RCOMP
- net /CPU_V1P8U_MEM renamed /CPU_V1P8U_MEM
- net /CPU_V1P8U_MEM_EDGECAP_0 renamed /CPU_V1P8U_MEM_EDGECAP_0
- net /CPU_V1P8U_MEM_EDGECAP_1 renamed /CPU_V1P8U_MEM_EDGECAP_1
- net /CPU_V1P8U_MEM_EDGECAP_2 renamed /CPU_V1P8U_MEM_EDGECAP_2
- net /CPU_V1P8U_MEM_EDGECAP_3 renamed /CPU_V1P8U_MEM_EDGECAP_3
- net /CPU_VCCGT renamed /CPU_VCCGT
- net /CPU_VCCGT_SENSE renamed /CPU_VCCGT_SENSE
- net /CPU_VCCGT_VSS_SENSE renamed /CPU_VCCGT_VSS_SENSE
- net /CPU_VCCL2 renamed /CPU_VCCL2
- net /CPU_VCCL2_SENSE renamed /CPU_VCCL2_SENSE
- net /CPU_VCCL2_VSS_SENSE renamed /CPU_VCCL2_VSS_SENSE
- net /CPU_VCCPRIM_1P8 renamed /CPU_VCCPRIM_1P8
- net /CPU_VCCPRIM_1P8_FLTRA_IN renamed /CPU_VCCPRIM_1P8_FLTRA_IN
- net /CPU_VCCPRIM_1P8_FLTRB_CAP renamed /CPU_VCCPRIM_1P8_FLTRB_CAP
- net /CPU_VCCPRIM_1P8_FLTRB_IN renamed /CPU_VCCPRIM_1P8_FLTRB_IN
- net /CPU_VCCPRIM_3P3 renamed /CPU_VCCPRIM_3P3
- net /CPU_VCCPRIM_IO renamed /CPU_VCCPRIM_IO
- net /CPU_VCCPRIM_IO_SENSE renamed /CPU_VCCPRIM_IO_SENSE
- net /CPU_VCCPRIM_IO_VSS_SENSE renamed /CPU_VCCPRIM_IO_VSS_SENSE
- net /CPU_VCCPRIM_VNNAON renamed /CPU_VCCPRIM_VNNAON
- net /CPU_VCCPRIM_VNNAONLV renamed /CPU_VCCPRIM_VNNAONLV
- net /CPU_VCCPRIM_VNNAONLV_SENSE renamed /CPU_VCCPRIM_VNNAONLV_SENSE
- net /CPU_VCCPRIM_VNNAONLV_VSS_SENSE renamed /CPU_VCCPRIM_VNNAONLV_VSS_SENSE
- net /CPU_VCCPRIM_VNNAON_FLTR renamed /CPU_VCCPRIM_VNNAON_FLTR
- net /CPU_VCCPRIM_VNNAON_SENSE renamed /CPU_VCCPRIM_VNNAON_SENSE
- net /CPU_VCCPRIM_VNNAON_VSS_SENSE renamed /CPU_VCCPRIM_VNNAON_VSS_SENSE
- net /CPU_VCCRTC renamed /CPU_VCCRTC
- net /CPU_VCCSA renamed /CPU_VCCSA
- net /CPU_VCCSA_SENSE renamed /CPU_VCCSA_SENSE
- net /CPU_VCCSA_VSS_SENSE renamed /CPU_VCCSA_VSS_SENSE
- net /CPU_VCCST renamed /CPU_VCCST
- net /CPU_VCCST_EN_1V8 renamed /CPU_VCCST_EN_1V8
- net /CPU_VCC_ECORE renamed /CPU_VCC_ECORE
- net /CPU_VCC_ECORE_SENSE renamed /CPU_VCC_ECORE_SENSE
- net /CPU_VCC_ECORE_VSS_SENSE renamed /CPU_VCC_ECORE_VSS_SENSE
- net /CPU_VCC_PCORE renamed /CPU_VCC_PCORE
- net /CPU_VCC_PCORE_SENSE renamed /CPU_VCC_PCORE_SENSE
- net /CPU_VCC_PCORE_VSS_SENSE renamed /CPU_VCC_PCORE_VSS_SENSE
- net /CPU_VDD2H renamed /CPU_VDD2H
- net /CPU_VDD2H_EDGECAP_0 renamed /CPU_VDD2H_EDGECAP_0
- net /CPU_VDD2H_EDGECAP_1 renamed /CPU_VDD2H_EDGECAP_1
- net /CPU_VDD2H_SENSE renamed /CPU_VDD2H_SENSE
- net /CPU_VDD2H_VSS_SENSE renamed /CPU_VDD2H_VSS_SENSE
- net /CPU_VDD2L renamed /CPU_VDD2L
- net /CPU_VDD2L_EDGECAP_0 renamed /CPU_VDD2L_EDGECAP_0
- net /CPU_VDD2L_EDGECAP_1 renamed /CPU_VDD2L_EDGECAP_1
- net /CPU_VDD2L_SENSE renamed /CPU_VDD2L_SENSE
- net /CPU_VDD2L_VSS_SENSE renamed /CPU_VDD2L_VSS_SENSE
- net /CPU_VDD2_PWRGOOD_LOOP renamed /CPU_VDD2_PWRGOOD_LOOP
- net /CPU_VDDQ renamed /CPU_VDDQ
- net /CPU_VDDQ_EDGECAP_0 renamed /CPU_VDDQ_EDGECAP_0
- net /CPU_VDDQ_EDGECAP_1 renamed /CPU_VDDQ_EDGECAP_1
- net /CPU_VDDQ_SENSE renamed /CPU_VDDQ_SENSE
- net /CPU_VDDQ_VSS_SENSE renamed /CPU_VDDQ_VSS_SENSE
- net /CPU_VDDRIO renamed /CPU_VDDRIO
- net /CPU_VDDRIO_SENSE renamed /CPU_VDDRIO_SENSE
- net /CPU_VDDRIO_VSS_SENSE renamed /CPU_VDDRIO_VSS_SENSE
- net /CPU_WAKE_N renamed /CPU_WAKE_N
- net /CPU_XTAL_IN renamed /CPU_XTAL_IN
- net /CPU_XTAL_OUT renamed /CPU_XTAL_OUT
- net /CUSTOM_12V_RAW renamed /CUSTOM_12V_RAW
- net /CUSTOM_DET_A renamed /CUSTOM_DET_A
- net /CUSTOM_DET_B renamed /CUSTOM_DET_B
- net /EXT_41_DVDT renamed /EXT_41_DVDT
- net /EXT_41_ILM renamed /EXT_41_ILM
- net /EXT_41_OV renamed /EXT_41_OV
- net /EXT_41_UV renamed /EXT_41_UV
- net /EXT_42_DVDT renamed /EXT_42_DVDT
- net /EXT_42_ILM renamed /EXT_42_ILM
- net /EXT_42_OV renamed /EXT_42_OV
- net /EXT_42_UV renamed /EXT_42_UV
- net /GND renamed /GND
- net /M1_3V3 renamed /M1_3V3
- net /M1_BST renamed /M1_BST
- net /M1_CLKREQ renamed /M1_CLKREQ
- net /M1_CLK_N renamed /M1_CLK_N
- net /M1_CLK_P renamed /M1_CLK_P
- net /M1_FB renamed /M1_FB
- net /M1_RX0_N renamed /M1_RX0_N
- net /M1_RX0_P renamed /M1_RX0_P
- net /M1_RX1_N renamed /M1_RX1_N
- net /M1_RX1_P renamed /M1_RX1_P
- net /M1_RX2_N renamed /M1_RX2_N
- net /M1_RX2_P renamed /M1_RX2_P
- net /M1_RX3_N renamed /M1_RX3_N
- net /M1_RX3_P renamed /M1_RX3_P
- net /M1_SW renamed /M1_SW
- net /M1_TX0_N renamed /M1_TX0_N
- net /M1_TX0_N_AC renamed /M1_TX0_N_AC
- net /M1_TX0_P renamed /M1_TX0_P
- net /M1_TX0_P_AC renamed /M1_TX0_P_AC
- net /M1_TX1_N renamed /M1_TX1_N
- net /M1_TX1_N_AC renamed /M1_TX1_N_AC
- net /M1_TX1_P renamed /M1_TX1_P
- net /M1_TX1_P_AC renamed /M1_TX1_P_AC
- net /M1_TX2_N renamed /M1_TX2_N
- net /M1_TX2_N_AC renamed /M1_TX2_N_AC
- net /M1_TX2_P renamed /M1_TX2_P
- net /M1_TX2_P_AC renamed /M1_TX2_P_AC
- net /M1_TX3_N renamed /M1_TX3_N
- net /M1_TX3_N_AC renamed /M1_TX3_N_AC
- net /M1_TX3_P renamed /M1_TX3_P
- net /M1_TX3_P_AC renamed /M1_TX3_P_AC
- net /M1_WAKE renamed /M1_WAKE
- net /M2_12V_L renamed /M2_12V_L
- net /M2_12V_R renamed /M2_12V_R
- net /M2_3V3 renamed /M2_3V3
- net /M2_BST renamed /M2_BST
- net /M2_CLKREQ renamed /M2_CLKREQ
- net /M2_CLK_N renamed /M2_CLK_N
- net /M2_CLK_P renamed /M2_CLK_P
- net /M2_FB renamed /M2_FB
- net /M2_RX0_N renamed /M2_RX0_N
- net /M2_RX0_P renamed /M2_RX0_P
- net /M2_RX1_N renamed /M2_RX1_N
- net /M2_RX1_P renamed /M2_RX1_P
- net /M2_RX2_N renamed /M2_RX2_N
- net /M2_RX2_P renamed /M2_RX2_P
- net /M2_RX3_N renamed /M2_RX3_N
- net /M2_RX3_P renamed /M2_RX3_P
- net /M2_SW renamed /M2_SW
- net /M2_TX0_N renamed /M2_TX0_N
- net /M2_TX0_N_AC renamed /M2_TX0_N_AC
- net /M2_TX0_P renamed /M2_TX0_P
- net /M2_TX0_P_AC renamed /M2_TX0_P_AC
- net /M2_TX1_N renamed /M2_TX1_N
- net /M2_TX1_N_AC renamed /M2_TX1_N_AC
- net /M2_TX1_P renamed /M2_TX1_P
- net /M2_TX1_P_AC renamed /M2_TX1_P_AC
- net /M2_TX2_N renamed /M2_TX2_N
- net /M2_TX2_N_AC renamed /M2_TX2_N_AC
- net /M2_TX2_P renamed /M2_TX2_P
- net /M2_TX2_P_AC renamed /M2_TX2_P_AC
- net /M2_TX3_N renamed /M2_TX3_N
- net /M2_TX3_N_AC renamed /M2_TX3_N_AC
- net /M2_TX3_P renamed /M2_TX3_P
- net /M2_TX3_P_AC renamed /M2_TX3_P_AC
- net /M2_WAKE renamed /M2_WAKE
- net /M3_3V3 renamed /M3_3V3
- net /M3_BST renamed /M3_BST
- net /M3_CLKREQ renamed /M3_CLKREQ
- net /M3_CLK_N renamed /M3_CLK_N
- net /M3_CLK_P renamed /M3_CLK_P
- net /M3_FB renamed /M3_FB
- net /M3_RX0_N renamed /M3_RX0_N
- net /M3_RX0_P renamed /M3_RX0_P
- net /M3_RX1_N renamed /M3_RX1_N
- net /M3_RX1_P renamed /M3_RX1_P
- net /M3_RX2_N renamed /M3_RX2_N
- net /M3_RX2_P renamed /M3_RX2_P
- net /M3_RX3_N renamed /M3_RX3_N
- net /M3_RX3_P renamed /M3_RX3_P
- net /M3_SW renamed /M3_SW
- net /M3_TX0_N renamed /M3_TX0_N
- net /M3_TX0_N_AC renamed /M3_TX0_N_AC
- net /M3_TX0_P renamed /M3_TX0_P
- net /M3_TX0_P_AC renamed /M3_TX0_P_AC
- net /M3_TX1_N renamed /M3_TX1_N
- net /M3_TX1_N_AC renamed /M3_TX1_N_AC
- net /M3_TX1_P renamed /M3_TX1_P
- net /M3_TX1_P_AC renamed /M3_TX1_P_AC
- net /M3_TX2_N renamed /M3_TX2_N
- net /M3_TX2_N_AC renamed /M3_TX2_N_AC
- net /M3_TX2_P renamed /M3_TX2_P
- net /M3_TX2_P_AC renamed /M3_TX2_P_AC
- net /M3_TX3_N renamed /M3_TX3_N
- net /M3_TX3_N_AC renamed /M3_TX3_N_AC
- net /M3_TX3_P renamed /M3_TX3_P
- net /M3_TX3_P_AC renamed /M3_TX3_P_AC
- net /M3_WAKE renamed /M3_WAKE
- net /M4_3V3 renamed /M4_3V3
- net /M4_BST renamed /M4_BST
- net /M4_CLKREQ renamed /M4_CLKREQ
- net /M4_CLK_N renamed /M4_CLK_N
- net /M4_CLK_P renamed /M4_CLK_P
- net /M4_FB renamed /M4_FB
- net /M4_RX0_N renamed /M4_RX0_N
- net /M4_RX0_P renamed /M4_RX0_P
- net /M4_RX1_N renamed /M4_RX1_N
- net /M4_RX1_P renamed /M4_RX1_P
- net /M4_RX2_N renamed /M4_RX2_N
- net /M4_RX2_P renamed /M4_RX2_P
- net /M4_RX3_N renamed /M4_RX3_N
- net /M4_RX3_P renamed /M4_RX3_P
- net /M4_SW renamed /M4_SW
- net /M4_TX0_N renamed /M4_TX0_N
- net /M4_TX0_N_AC renamed /M4_TX0_N_AC
- net /M4_TX0_P renamed /M4_TX0_P
- net /M4_TX0_P_AC renamed /M4_TX0_P_AC
- net /M4_TX1_N renamed /M4_TX1_N
- net /M4_TX1_N_AC renamed /M4_TX1_N_AC
- net /M4_TX1_P renamed /M4_TX1_P
- net /M4_TX1_P_AC renamed /M4_TX1_P_AC
- net /M4_TX2_N renamed /M4_TX2_N
- net /M4_TX2_N_AC renamed /M4_TX2_N_AC
- net /M4_TX2_P renamed /M4_TX2_P
- net /M4_TX2_P_AC renamed /M4_TX2_P_AC
- net /M4_TX3_N renamed /M4_TX3_N
- net /M4_TX3_N_AC renamed /M4_TX3_N_AC
- net /M4_TX3_P renamed /M4_TX3_P
- net /M4_TX3_P_AC renamed /M4_TX3_P_AC
- net /M4_WAKE renamed /M4_WAKE
- net /N01_3V3 renamed /N01_3V3
- net /N01_CLKREQ renamed /N01_CLKREQ
- net /N01_CLK_N renamed /N01_CLK_N
- net /N01_CLK_P renamed /N01_CLK_P
- net /N01_FB renamed /N01_FB
- net /N01_PERST renamed /N01_PERST
- net /N01_RX0_N renamed /N01_RX0_N
- net /N01_RX0_P renamed /N01_RX0_P
- net /N01_RX1_N renamed /N01_RX1_N
- net /N01_RX1_P renamed /N01_RX1_P
- net /N01_RX2_N renamed /N01_RX2_N
- net /N01_RX2_P renamed /N01_RX2_P
- net /N01_RX3_N renamed /N01_RX3_N
- net /N01_RX3_P renamed /N01_RX3_P
- net /N01_TX0_N renamed /N01_TX0_N
- net /N01_TX0_N_AC renamed /N01_TX0_N_AC
- net /N01_TX0_P renamed /N01_TX0_P
- net /N01_TX0_P_AC renamed /N01_TX0_P_AC
- net /N01_TX1_N renamed /N01_TX1_N
- net /N01_TX1_N_AC renamed /N01_TX1_N_AC
- net /N01_TX1_P renamed /N01_TX1_P
- net /N01_TX1_P_AC renamed /N01_TX1_P_AC
- net /N01_TX2_N renamed /N01_TX2_N
- net /N01_TX2_N_AC renamed /N01_TX2_N_AC
- net /N01_TX2_P renamed /N01_TX2_P
- net /N01_TX2_P_AC renamed /N01_TX2_P_AC
- net /N01_TX3_N renamed /N01_TX3_N
- net /N01_TX3_N_AC renamed /N01_TX3_N_AC
- net /N01_TX3_P renamed /N01_TX3_P
- net /N01_TX3_P_AC renamed /N01_TX3_P_AC
- net /N01_WAKE renamed /N01_WAKE
- net /N02_3V3 renamed /N02_3V3
- net /N02_CLKREQ renamed /N02_CLKREQ
- net /N02_CLK_N renamed /N02_CLK_N
- net /N02_CLK_P renamed /N02_CLK_P
- net /N02_FB renamed /N02_FB
- net /N02_PERST renamed /N02_PERST
- net /N02_RX0_N renamed /N02_RX0_N
- net /N02_RX0_P renamed /N02_RX0_P
- net /N02_RX1_N renamed /N02_RX1_N
- net /N02_RX1_P renamed /N02_RX1_P
- net /N02_RX2_N renamed /N02_RX2_N
- net /N02_RX2_P renamed /N02_RX2_P
- net /N02_RX3_N renamed /N02_RX3_N
- net /N02_RX3_P renamed /N02_RX3_P
- net /N02_TX0_N renamed /N02_TX0_N
- net /N02_TX0_N_AC renamed /N02_TX0_N_AC
- net /N02_TX0_P renamed /N02_TX0_P
- net /N02_TX0_P_AC renamed /N02_TX0_P_AC
- net /N02_TX1_N renamed /N02_TX1_N
- net /N02_TX1_N_AC renamed /N02_TX1_N_AC
- net /N02_TX1_P renamed /N02_TX1_P
- net /N02_TX1_P_AC renamed /N02_TX1_P_AC
- net /N02_TX2_N renamed /N02_TX2_N
- net /N02_TX2_N_AC renamed /N02_TX2_N_AC
- net /N02_TX2_P renamed /N02_TX2_P
- net /N02_TX2_P_AC renamed /N02_TX2_P_AC
- net /N02_TX3_N renamed /N02_TX3_N
- net /N02_TX3_N_AC renamed /N02_TX3_N_AC
- net /N02_TX3_P renamed /N02_TX3_P
- net /N02_TX3_P_AC renamed /N02_TX3_P_AC
- net /N02_WAKE renamed /N02_WAKE
- net /N03_3V3 renamed /N03_3V3
- net /N03_CLKREQ renamed /N03_CLKREQ
- net /N03_CLK_N renamed /N03_CLK_N
- net /N03_CLK_P renamed /N03_CLK_P
- net /N03_FB renamed /N03_FB
- net /N03_PERST renamed /N03_PERST
- net /N03_RX0_N renamed /N03_RX0_N
- net /N03_RX0_P renamed /N03_RX0_P
- net /N03_RX1_N renamed /N03_RX1_N
- net /N03_RX1_P renamed /N03_RX1_P
- net /N03_RX2_N renamed /N03_RX2_N
- net /N03_RX2_P renamed /N03_RX2_P
- net /N03_RX3_N renamed /N03_RX3_N
- net /N03_RX3_P renamed /N03_RX3_P
- net /N03_TX0_N renamed /N03_TX0_N
- net /N03_TX0_N_AC renamed /N03_TX0_N_AC
- net /N03_TX0_P renamed /N03_TX0_P
- net /N03_TX0_P_AC renamed /N03_TX0_P_AC
- net /N03_TX1_N renamed /N03_TX1_N
- net /N03_TX1_N_AC renamed /N03_TX1_N_AC
- net /N03_TX1_P renamed /N03_TX1_P
- net /N03_TX1_P_AC renamed /N03_TX1_P_AC
- net /N03_TX2_N renamed /N03_TX2_N
- net /N03_TX2_N_AC renamed /N03_TX2_N_AC
- net /N03_TX2_P renamed /N03_TX2_P
- net /N03_TX2_P_AC renamed /N03_TX2_P_AC
- net /N03_TX3_N renamed /N03_TX3_N
- net /N03_TX3_N_AC renamed /N03_TX3_N_AC
- net /N03_TX3_P renamed /N03_TX3_P
- net /N03_TX3_P_AC renamed /N03_TX3_P_AC
- net /N03_WAKE renamed /N03_WAKE
- net /N04_3V3 renamed /N04_3V3
- net /N04_CLKREQ renamed /N04_CLKREQ
- net /N04_CLK_N renamed /N04_CLK_N
- net /N04_CLK_P renamed /N04_CLK_P
- net /N04_FB renamed /N04_FB
- net /N04_PERST renamed /N04_PERST
- net /N04_RX0_N renamed /N04_RX0_N
- net /N04_RX0_P renamed /N04_RX0_P
- net /N04_RX1_N renamed /N04_RX1_N
- net /N04_RX1_P renamed /N04_RX1_P
- net /N04_RX2_N renamed /N04_RX2_N
- net /N04_RX2_P renamed /N04_RX2_P
- net /N04_RX3_N renamed /N04_RX3_N
- net /N04_RX3_P renamed /N04_RX3_P
- net /N04_TX0_N renamed /N04_TX0_N
- net /N04_TX0_N_AC renamed /N04_TX0_N_AC
- net /N04_TX0_P renamed /N04_TX0_P
- net /N04_TX0_P_AC renamed /N04_TX0_P_AC
- net /N04_TX1_N renamed /N04_TX1_N
- net /N04_TX1_N_AC renamed /N04_TX1_N_AC
- net /N04_TX1_P renamed /N04_TX1_P
- net /N04_TX1_P_AC renamed /N04_TX1_P_AC
- net /N04_TX2_N renamed /N04_TX2_N
- net /N04_TX2_N_AC renamed /N04_TX2_N_AC
- net /N04_TX2_P renamed /N04_TX2_P
- net /N04_TX2_P_AC renamed /N04_TX2_P_AC
- net /N04_TX3_N renamed /N04_TX3_N
- net /N04_TX3_N_AC renamed /N04_TX3_N_AC
- net /N04_TX3_P renamed /N04_TX3_P
- net /N04_TX3_P_AC renamed /N04_TX3_P_AC
- net /N04_WAKE renamed /N04_WAKE
- net /N05_3V3 renamed /N05_3V3
- net /N05_CLKREQ renamed /N05_CLKREQ
- net /N05_CLK_N renamed /N05_CLK_N
- net /N05_CLK_P renamed /N05_CLK_P
- net /N05_FB renamed /N05_FB
- net /N05_PERST renamed /N05_PERST
- net /N05_RX0_N renamed /N05_RX0_N
- net /N05_RX0_P renamed /N05_RX0_P
- net /N05_RX1_N renamed /N05_RX1_N
- net /N05_RX1_P renamed /N05_RX1_P
- net /N05_RX2_N renamed /N05_RX2_N
- net /N05_RX2_P renamed /N05_RX2_P
- net /N05_RX3_N renamed /N05_RX3_N
- net /N05_RX3_P renamed /N05_RX3_P
- net /N05_TX0_N renamed /N05_TX0_N
- net /N05_TX0_N_AC renamed /N05_TX0_N_AC
- net /N05_TX0_P renamed /N05_TX0_P
- net /N05_TX0_P_AC renamed /N05_TX0_P_AC
- net /N05_TX1_N renamed /N05_TX1_N
- net /N05_TX1_N_AC renamed /N05_TX1_N_AC
- net /N05_TX1_P renamed /N05_TX1_P
- net /N05_TX1_P_AC renamed /N05_TX1_P_AC
- net /N05_TX2_N renamed /N05_TX2_N
- net /N05_TX2_N_AC renamed /N05_TX2_N_AC
- net /N05_TX2_P renamed /N05_TX2_P
- net /N05_TX2_P_AC renamed /N05_TX2_P_AC
- net /N05_TX3_N renamed /N05_TX3_N
- net /N05_TX3_N_AC renamed /N05_TX3_N_AC
- net /N05_TX3_P renamed /N05_TX3_P
- net /N05_TX3_P_AC renamed /N05_TX3_P_AC
- net /N05_WAKE renamed /N05_WAKE
- net /N06_3V3 renamed /N06_3V3
- net /N06_CLKREQ renamed /N06_CLKREQ
- net /N06_CLK_N renamed /N06_CLK_N
- net /N06_CLK_P renamed /N06_CLK_P
- net /N06_FB renamed /N06_FB
- net /N06_PERST renamed /N06_PERST
- net /N06_RX0_N renamed /N06_RX0_N
- net /N06_RX0_P renamed /N06_RX0_P
- net /N06_RX1_N renamed /N06_RX1_N
- net /N06_RX1_P renamed /N06_RX1_P
- net /N06_RX2_N renamed /N06_RX2_N
- net /N06_RX2_P renamed /N06_RX2_P
- net /N06_RX3_N renamed /N06_RX3_N
- net /N06_RX3_P renamed /N06_RX3_P
- net /N06_TX0_N renamed /N06_TX0_N
- net /N06_TX0_N_AC renamed /N06_TX0_N_AC
- net /N06_TX0_P renamed /N06_TX0_P
- net /N06_TX0_P_AC renamed /N06_TX0_P_AC
- net /N06_TX1_N renamed /N06_TX1_N
- net /N06_TX1_N_AC renamed /N06_TX1_N_AC
- net /N06_TX1_P renamed /N06_TX1_P
- net /N06_TX1_P_AC renamed /N06_TX1_P_AC
- net /N06_TX2_N renamed /N06_TX2_N
- net /N06_TX2_N_AC renamed /N06_TX2_N_AC
- net /N06_TX2_P renamed /N06_TX2_P
- net /N06_TX2_P_AC renamed /N06_TX2_P_AC
- net /N06_TX3_N renamed /N06_TX3_N
- net /N06_TX3_N_AC renamed /N06_TX3_N_AC
- net /N06_TX3_P renamed /N06_TX3_P
- net /N06_TX3_P_AC renamed /N06_TX3_P_AC
- net /N06_WAKE renamed /N06_WAKE
- net /N07_3V3 renamed /N07_3V3
- net /N07_CLKREQ renamed /N07_CLKREQ
- net /N07_CLK_N renamed /N07_CLK_N
- net /N07_CLK_P renamed /N07_CLK_P
- net /N07_FB renamed /N07_FB
- net /N07_PERST renamed /N07_PERST
- net /N07_RX0_N renamed /N07_RX0_N
- net /N07_RX0_P renamed /N07_RX0_P
- net /N07_RX1_N renamed /N07_RX1_N
- net /N07_RX1_P renamed /N07_RX1_P
- net /N07_RX2_N renamed /N07_RX2_N
- net /N07_RX2_P renamed /N07_RX2_P
- net /N07_RX3_N renamed /N07_RX3_N
- net /N07_RX3_P renamed /N07_RX3_P
- net /N07_TX0_N renamed /N07_TX0_N
- net /N07_TX0_N_AC renamed /N07_TX0_N_AC
- net /N07_TX0_P renamed /N07_TX0_P
- net /N07_TX0_P_AC renamed /N07_TX0_P_AC
- net /N07_TX1_N renamed /N07_TX1_N
- net /N07_TX1_N_AC renamed /N07_TX1_N_AC
- net /N07_TX1_P renamed /N07_TX1_P
- net /N07_TX1_P_AC renamed /N07_TX1_P_AC
- net /N07_TX2_N renamed /N07_TX2_N
- net /N07_TX2_N_AC renamed /N07_TX2_N_AC
- net /N07_TX2_P renamed /N07_TX2_P
- net /N07_TX2_P_AC renamed /N07_TX2_P_AC
- net /N07_TX3_N renamed /N07_TX3_N
- net /N07_TX3_N_AC renamed /N07_TX3_N_AC
- net /N07_TX3_P renamed /N07_TX3_P
- net /N07_TX3_P_AC renamed /N07_TX3_P_AC
- net /N07_WAKE renamed /N07_WAKE
- net /N08_3V3 renamed /N08_3V3
- net /N08_CLKREQ renamed /N08_CLKREQ
- net /N08_CLK_N renamed /N08_CLK_N
- net /N08_CLK_P renamed /N08_CLK_P
- net /N08_FB renamed /N08_FB
- net /N08_PERST renamed /N08_PERST
- net /N08_RX0_N renamed /N08_RX0_N
- net /N08_RX0_P renamed /N08_RX0_P
- net /N08_RX1_N renamed /N08_RX1_N
- net /N08_RX1_P renamed /N08_RX1_P
- net /N08_RX2_N renamed /N08_RX2_N
- net /N08_RX2_P renamed /N08_RX2_P
- net /N08_RX3_N renamed /N08_RX3_N
- net /N08_RX3_P renamed /N08_RX3_P
- net /N08_TX0_N renamed /N08_TX0_N
- net /N08_TX0_N_AC renamed /N08_TX0_N_AC
- net /N08_TX0_P renamed /N08_TX0_P
- net /N08_TX0_P_AC renamed /N08_TX0_P_AC
- net /N08_TX1_N renamed /N08_TX1_N
- net /N08_TX1_N_AC renamed /N08_TX1_N_AC
- net /N08_TX1_P renamed /N08_TX1_P
- net /N08_TX1_P_AC renamed /N08_TX1_P_AC
- net /N08_TX2_N renamed /N08_TX2_N
- net /N08_TX2_N_AC renamed /N08_TX2_N_AC
- net /N08_TX2_P renamed /N08_TX2_P
- net /N08_TX2_P_AC renamed /N08_TX2_P_AC
- net /N08_TX3_N renamed /N08_TX3_N
- net /N08_TX3_N_AC renamed /N08_TX3_N_AC
- net /N08_TX3_P renamed /N08_TX3_P
- net /N08_TX3_P_AC renamed /N08_TX3_P_AC
- net /N08_WAKE renamed /N08_WAKE
- net /N09_3V3 renamed /N09_3V3
- net /N09_CLKREQ renamed /N09_CLKREQ
- net /N09_CLK_N renamed /N09_CLK_N
- net /N09_CLK_P renamed /N09_CLK_P
- net /N09_FB renamed /N09_FB
- net /N09_PERST renamed /N09_PERST
- net /N09_RX0_N renamed /N09_RX0_N
- net /N09_RX0_P renamed /N09_RX0_P
- net /N09_RX1_N renamed /N09_RX1_N
- net /N09_RX1_P renamed /N09_RX1_P
- net /N09_RX2_N renamed /N09_RX2_N
- net /N09_RX2_P renamed /N09_RX2_P
- net /N09_RX3_N renamed /N09_RX3_N
- net /N09_RX3_P renamed /N09_RX3_P
- net /N09_TX0_N renamed /N09_TX0_N
- net /N09_TX0_N_AC renamed /N09_TX0_N_AC
- net /N09_TX0_P renamed /N09_TX0_P
- net /N09_TX0_P_AC renamed /N09_TX0_P_AC
- net /N09_TX1_N renamed /N09_TX1_N
- net /N09_TX1_N_AC renamed /N09_TX1_N_AC
- net /N09_TX1_P renamed /N09_TX1_P
- net /N09_TX1_P_AC renamed /N09_TX1_P_AC
- net /N09_TX2_N renamed /N09_TX2_N
- net /N09_TX2_N_AC renamed /N09_TX2_N_AC
- net /N09_TX2_P renamed /N09_TX2_P
- net /N09_TX2_P_AC renamed /N09_TX2_P_AC
- net /N09_TX3_N renamed /N09_TX3_N
- net /N09_TX3_N_AC renamed /N09_TX3_N_AC
- net /N09_TX3_P renamed /N09_TX3_P
- net /N09_TX3_P_AC renamed /N09_TX3_P_AC
- net /N09_WAKE renamed /N09_WAKE
- net /N10_3V3 renamed /N10_3V3
- net /N10_CLKREQ renamed /N10_CLKREQ
- net /N10_CLK_N renamed /N10_CLK_N
- net /N10_CLK_P renamed /N10_CLK_P
- net /N10_FB renamed /N10_FB
- net /N10_PERST renamed /N10_PERST
- net /N10_RX0_N renamed /N10_RX0_N
- net /N10_RX0_P renamed /N10_RX0_P
- net /N10_RX1_N renamed /N10_RX1_N
- net /N10_RX1_P renamed /N10_RX1_P
- net /N10_RX2_N renamed /N10_RX2_N
- net /N10_RX2_P renamed /N10_RX2_P
- net /N10_RX3_N renamed /N10_RX3_N
- net /N10_RX3_P renamed /N10_RX3_P
- net /N10_TX0_N renamed /N10_TX0_N
- net /N10_TX0_N_AC renamed /N10_TX0_N_AC
- net /N10_TX0_P renamed /N10_TX0_P
- net /N10_TX0_P_AC renamed /N10_TX0_P_AC
- net /N10_TX1_N renamed /N10_TX1_N
- net /N10_TX1_N_AC renamed /N10_TX1_N_AC
- net /N10_TX1_P renamed /N10_TX1_P
- net /N10_TX1_P_AC renamed /N10_TX1_P_AC
- net /N10_TX2_N renamed /N10_TX2_N
- net /N10_TX2_N_AC renamed /N10_TX2_N_AC
- net /N10_TX2_P renamed /N10_TX2_P
- net /N10_TX2_P_AC renamed /N10_TX2_P_AC
- net /N10_TX3_N renamed /N10_TX3_N
- net /N10_TX3_N_AC renamed /N10_TX3_N_AC
- net /N10_TX3_P renamed /N10_TX3_P
- net /N10_TX3_P_AC renamed /N10_TX3_P_AC
- net /N10_WAKE renamed /N10_WAKE
- net /N11_3V3 renamed /N11_3V3
- net /N11_CLKREQ renamed /N11_CLKREQ
- net /N11_CLK_N renamed /N11_CLK_N
- net /N11_CLK_P renamed /N11_CLK_P
- net /N11_FB renamed /N11_FB
- net /N11_PERST renamed /N11_PERST
- net /N11_RX0_N renamed /N11_RX0_N
- net /N11_RX0_P renamed /N11_RX0_P
- net /N11_RX1_N renamed /N11_RX1_N
- net /N11_RX1_P renamed /N11_RX1_P
- net /N11_RX2_N renamed /N11_RX2_N
- net /N11_RX2_P renamed /N11_RX2_P
- net /N11_RX3_N renamed /N11_RX3_N
- net /N11_RX3_P renamed /N11_RX3_P
- net /N11_TX0_N renamed /N11_TX0_N
- net /N11_TX0_N_AC renamed /N11_TX0_N_AC
- net /N11_TX0_P renamed /N11_TX0_P
- net /N11_TX0_P_AC renamed /N11_TX0_P_AC
- net /N11_TX1_N renamed /N11_TX1_N
- net /N11_TX1_N_AC renamed /N11_TX1_N_AC
- net /N11_TX1_P renamed /N11_TX1_P
- net /N11_TX1_P_AC renamed /N11_TX1_P_AC
- net /N11_TX2_N renamed /N11_TX2_N
- net /N11_TX2_N_AC renamed /N11_TX2_N_AC
- net /N11_TX2_P renamed /N11_TX2_P
- net /N11_TX2_P_AC renamed /N11_TX2_P_AC
- net /N11_TX3_N renamed /N11_TX3_N
- net /N11_TX3_N_AC renamed /N11_TX3_N_AC
- net /N11_TX3_P renamed /N11_TX3_P
- net /N11_TX3_P_AC renamed /N11_TX3_P_AC
- net /N11_WAKE renamed /N11_WAKE
- net /N12_3V3 renamed /N12_3V3
- net /N12_CLKREQ renamed /N12_CLKREQ
- net /N12_CLK_N renamed /N12_CLK_N
- net /N12_CLK_P renamed /N12_CLK_P
- net /N12_FB renamed /N12_FB
- net /N12_PERST renamed /N12_PERST
- net /N12_RX0_N renamed /N12_RX0_N
- net /N12_RX0_P renamed /N12_RX0_P
- net /N12_RX1_N renamed /N12_RX1_N
- net /N12_RX1_P renamed /N12_RX1_P
- net /N12_RX2_N renamed /N12_RX2_N
- net /N12_RX2_P renamed /N12_RX2_P
- net /N12_RX3_N renamed /N12_RX3_N
- net /N12_RX3_P renamed /N12_RX3_P
- net /N12_TX0_N renamed /N12_TX0_N
- net /N12_TX0_N_AC renamed /N12_TX0_N_AC
- net /N12_TX0_P renamed /N12_TX0_P
- net /N12_TX0_P_AC renamed /N12_TX0_P_AC
- net /N12_TX1_N renamed /N12_TX1_N
- net /N12_TX1_N_AC renamed /N12_TX1_N_AC
- net /N12_TX1_P renamed /N12_TX1_P
- net /N12_TX1_P_AC renamed /N12_TX1_P_AC
- net /N12_TX2_N renamed /N12_TX2_N
- net /N12_TX2_N_AC renamed /N12_TX2_N_AC
- net /N12_TX2_P renamed /N12_TX2_P
- net /N12_TX2_P_AC renamed /N12_TX2_P_AC
- net /N12_TX3_N renamed /N12_TX3_N
- net /N12_TX3_N_AC renamed /N12_TX3_N_AC
- net /N12_TX3_P renamed /N12_TX3_P
- net /N12_TX3_P_AC renamed /N12_TX3_P_AC
- net /N12_WAKE renamed /N12_WAKE
- net /N13_3V3 renamed /N13_3V3
- net /N13_CLKREQ renamed /N13_CLKREQ
- net /N13_CLK_N renamed /N13_CLK_N
- net /N13_CLK_P renamed /N13_CLK_P
- net /N13_FB renamed /N13_FB
- net /N13_PERST renamed /N13_PERST
- net /N13_RX0_N renamed /N13_RX0_N
- net /N13_RX0_P renamed /N13_RX0_P
- net /N13_RX1_N renamed /N13_RX1_N
- net /N13_RX1_P renamed /N13_RX1_P
- net /N13_RX2_N renamed /N13_RX2_N
- net /N13_RX2_P renamed /N13_RX2_P
- net /N13_RX3_N renamed /N13_RX3_N
- net /N13_RX3_P renamed /N13_RX3_P
- net /N13_TX0_N renamed /N13_TX0_N
- net /N13_TX0_N_AC renamed /N13_TX0_N_AC
- net /N13_TX0_P renamed /N13_TX0_P
- net /N13_TX0_P_AC renamed /N13_TX0_P_AC
- net /N13_TX1_N renamed /N13_TX1_N
- net /N13_TX1_N_AC renamed /N13_TX1_N_AC
- net /N13_TX1_P renamed /N13_TX1_P
- net /N13_TX1_P_AC renamed /N13_TX1_P_AC
- net /N13_TX2_N renamed /N13_TX2_N
- net /N13_TX2_N_AC renamed /N13_TX2_N_AC
- net /N13_TX2_P renamed /N13_TX2_P
- net /N13_TX2_P_AC renamed /N13_TX2_P_AC
- net /N13_TX3_N renamed /N13_TX3_N
- net /N13_TX3_N_AC renamed /N13_TX3_N_AC
- net /N13_TX3_P renamed /N13_TX3_P
- net /N13_TX3_P_AC renamed /N13_TX3_P_AC
- net /N13_WAKE renamed /N13_WAKE
- net /N14_3V3 renamed /N14_3V3
- net /N14_CLKREQ renamed /N14_CLKREQ
- net /N14_CLK_N renamed /N14_CLK_N
- net /N14_CLK_P renamed /N14_CLK_P
- net /N14_FB renamed /N14_FB
- net /N14_PERST renamed /N14_PERST
- net /N14_RX0_N renamed /N14_RX0_N
- net /N14_RX0_P renamed /N14_RX0_P
- net /N14_RX1_N renamed /N14_RX1_N
- net /N14_RX1_P renamed /N14_RX1_P
- net /N14_RX2_N renamed /N14_RX2_N
- net /N14_RX2_P renamed /N14_RX2_P
- net /N14_RX3_N renamed /N14_RX3_N
- net /N14_RX3_P renamed /N14_RX3_P
- net /N14_TX0_N renamed /N14_TX0_N
- net /N14_TX0_N_AC renamed /N14_TX0_N_AC
- net /N14_TX0_P renamed /N14_TX0_P
- net /N14_TX0_P_AC renamed /N14_TX0_P_AC
- net /N14_TX1_N renamed /N14_TX1_N
- net /N14_TX1_N_AC renamed /N14_TX1_N_AC
- net /N14_TX1_P renamed /N14_TX1_P
- net /N14_TX1_P_AC renamed /N14_TX1_P_AC
- net /N14_TX2_N renamed /N14_TX2_N
- net /N14_TX2_N_AC renamed /N14_TX2_N_AC
- net /N14_TX2_P renamed /N14_TX2_P
- net /N14_TX2_P_AC renamed /N14_TX2_P_AC
- net /N14_TX3_N renamed /N14_TX3_N
- net /N14_TX3_N_AC renamed /N14_TX3_N_AC
- net /N14_TX3_P renamed /N14_TX3_P
- net /N14_TX3_P_AC renamed /N14_TX3_P_AC
- net /N14_WAKE renamed /N14_WAKE
- net /N15_3V3 renamed /N15_3V3
- net /N15_CLKREQ renamed /N15_CLKREQ
- net /N15_CLK_N renamed /N15_CLK_N
- net /N15_CLK_P renamed /N15_CLK_P
- net /N15_FB renamed /N15_FB
- net /N15_PERST renamed /N15_PERST
- net /N15_RX0_N renamed /N15_RX0_N
- net /N15_RX0_P renamed /N15_RX0_P
- net /N15_RX1_N renamed /N15_RX1_N
- net /N15_RX1_P renamed /N15_RX1_P
- net /N15_RX2_N renamed /N15_RX2_N
- net /N15_RX2_P renamed /N15_RX2_P
- net /N15_RX3_N renamed /N15_RX3_N
- net /N15_RX3_P renamed /N15_RX3_P
- net /N15_TX0_N renamed /N15_TX0_N
- net /N15_TX0_N_AC renamed /N15_TX0_N_AC
- net /N15_TX0_P renamed /N15_TX0_P
- net /N15_TX0_P_AC renamed /N15_TX0_P_AC
- net /N15_TX1_N renamed /N15_TX1_N
- net /N15_TX1_N_AC renamed /N15_TX1_N_AC
- net /N15_TX1_P renamed /N15_TX1_P
- net /N15_TX1_P_AC renamed /N15_TX1_P_AC
- net /N15_TX2_N renamed /N15_TX2_N
- net /N15_TX2_N_AC renamed /N15_TX2_N_AC
- net /N15_TX2_P renamed /N15_TX2_P
- net /N15_TX2_P_AC renamed /N15_TX2_P_AC
- net /N15_TX3_N renamed /N15_TX3_N
- net /N15_TX3_N_AC renamed /N15_TX3_N_AC
- net /N15_TX3_P renamed /N15_TX3_P
- net /N15_TX3_P_AC renamed /N15_TX3_P_AC
- net /N15_WAKE renamed /N15_WAKE
- net /N16_3V3 renamed /N16_3V3
- net /N16_CLKREQ renamed /N16_CLKREQ
- net /N16_CLK_N renamed /N16_CLK_N
- net /N16_CLK_P renamed /N16_CLK_P
- net /N16_FB renamed /N16_FB
- net /N16_PERST renamed /N16_PERST
- net /N16_RX0_N renamed /N16_RX0_N
- net /N16_RX0_P renamed /N16_RX0_P
- net /N16_RX1_N renamed /N16_RX1_N
- net /N16_RX1_P renamed /N16_RX1_P
- net /N16_RX2_N renamed /N16_RX2_N
- net /N16_RX2_P renamed /N16_RX2_P
- net /N16_RX3_N renamed /N16_RX3_N
- net /N16_RX3_P renamed /N16_RX3_P
- net /N16_TX0_N renamed /N16_TX0_N
- net /N16_TX0_N_AC renamed /N16_TX0_N_AC
- net /N16_TX0_P renamed /N16_TX0_P
- net /N16_TX0_P_AC renamed /N16_TX0_P_AC
- net /N16_TX1_N renamed /N16_TX1_N
- net /N16_TX1_N_AC renamed /N16_TX1_N_AC
- net /N16_TX1_P renamed /N16_TX1_P
- net /N16_TX1_P_AC renamed /N16_TX1_P_AC
- net /N16_TX2_N renamed /N16_TX2_N
- net /N16_TX2_N_AC renamed /N16_TX2_N_AC
- net /N16_TX2_P renamed /N16_TX2_P
- net /N16_TX2_P_AC renamed /N16_TX2_P_AC
- net /N16_TX3_N renamed /N16_TX3_N
- net /N16_TX3_N_AC renamed /N16_TX3_N_AC
- net /N16_TX3_P renamed /N16_TX3_P
- net /N16_TX3_P_AC renamed /N16_TX3_P_AC
- net /N16_WAKE renamed /N16_WAKE
- net /P3V3_AUX renamed /P3V3_AUX
- net /PEX_0V9 renamed /PEX_0V9
- net /PEX_0V9A renamed /PEX_0V9A
- net /PEX_1V8 renamed /PEX_1V8
- net /PEX_1V8A renamed /PEX_1V8A
- net /PEX_MGMT_SCL_1V8 renamed /PEX_MGMT_SCL_1V8
- net /PEX_MGMT_SDA_1V8 renamed /PEX_MGMT_SDA_1V8
- net /PEX_RESET_CT renamed /PEX_RESET_CT
- net /PEX_SPI_CLK renamed /PEX_SPI_CLK
- net /PEX_SPI_CS_N renamed /PEX_SPI_CS_N
- net /PEX_SPI_IO0 renamed /PEX_SPI_IO0
- net /PEX_SPI_IO1 renamed /PEX_SPI_IO1
- net /PEX_SPI_IO2 renamed /PEX_SPI_IO2
- net /PEX_SPI_IO3 renamed /PEX_SPI_IO3
- net /PEX_SPI_RESET_N renamed /PEX_SPI_RESET_N
- net /PEX_STRAP_DBG_MODE0 renamed /PEX_STRAP_DBG_MODE0
- net /PEX_STRAP_DBG_MODE1 renamed /PEX_STRAP_DBG_MODE1
- net /PEX_STRAP_DBG_MODE2 renamed /PEX_STRAP_DBG_MODE2
- net /PEX_STRAP_DBG_MODE3 renamed /PEX_STRAP_DBG_MODE3
- net /PEX_STRAP_DFT_IDDT renamed /PEX_STRAP_DFT_IDDT
- net /PEX_STRAP_DFT_SCAN_ENABLE renamed /PEX_STRAP_DFT_SCAN_ENABLE
- net /PEX_STRAP_DFT_SHIFT_CLK renamed /PEX_STRAP_DFT_SHIFT_CLK
- net /PEX_STRAP_DFT_TN renamed /PEX_STRAP_DFT_TN
- net /PEX_STRAP_MODE_SEL0 renamed /PEX_STRAP_MODE_SEL0
- net /PEX_STRAP_MODE_SEL1 renamed /PEX_STRAP_MODE_SEL1
- net /PEX_STRAP_MODE_SEL2 renamed /PEX_STRAP_MODE_SEL2
- net /PEX_STRAP_MODE_SEL3 renamed /PEX_STRAP_MODE_SEL3
- net /PEX_STRAP_MODE_SEL4 renamed /PEX_STRAP_MODE_SEL4
- net /PEX_STRAP_MODE_SEL5 renamed /PEX_STRAP_MODE_SEL5
- net /PEX_STRAP_MODE_SEL6 renamed /PEX_STRAP_MODE_SEL6
- net /PEX_STRAP_MODE_SEL7 renamed /PEX_STRAP_MODE_SEL7
- net /PEX_STRAP_MODE_SEL8 renamed /PEX_STRAP_MODE_SEL8
- net /PEX_STRAP_TRST_L renamed /PEX_STRAP_TRST_L
- net /PEX_SYS_REFCLK_N renamed /PEX_SYS_REFCLK_N
- net /PEX_SYS_REFCLK_P renamed /PEX_SYS_REFCLK_P
- net /PEX_SYS_RESET_N renamed /PEX_SYS_RESET_N
- net /REF_KA_DIF0N renamed /REF_KA_DIF0N
- net /REF_KA_DIF0P renamed /REF_KA_DIF0P
- net /REF_KA_OE1 renamed /REF_KA_OE1
- net /REF_KA_PD# renamed /REF_KA_PD#
- net /REF_KA_SSEN renamed /REF_KA_SSEN
- net /REF_KA_VDD renamed /REF_KA_VDD
- net /REF_KA_VDDA renamed /REF_KA_VDDA
- net /REF_KA_X1 renamed /REF_KA_X1
- net /REF_KA_X2 renamed /REF_KA_X2
- net /REF_KB_DIF0N renamed /REF_KB_DIF0N
- net /REF_KB_DIF0P renamed /REF_KB_DIF0P
- net /REF_KB_DIF1N renamed /REF_KB_DIF1N
- net /REF_KB_DIF1P renamed /REF_KB_DIF1P
- net /REF_KB_DIF2N renamed /REF_KB_DIF2N
- net /REF_KB_DIF2P renamed /REF_KB_DIF2P
- net /REF_KB_DIF3N renamed /REF_KB_DIF3N
- net /REF_KB_DIF3P renamed /REF_KB_DIF3P
- net /REF_KB_MODE renamed /REF_KB_MODE
- net /REF_KB_SELAB renamed /REF_KB_SELAB
- net /REF_KB_VDD renamed /REF_KB_VDD
- net /REF_KB_VDDA renamed /REF_KB_VDDA
- net /REF_KB_VDDB renamed /REF_KB_VDDB
- net /REF_PERST_BUFF# renamed /REF_PERST_BUFF#
- net /REF_PE_REFCLKN renamed /REF_PE_REFCLKN
- net /REF_PE_REFCLKP renamed /REF_PE_REFCLKP
- net /REF_SLIMA0_CLK renamed /REF_SLIMA0_CLK
- net /REF_SLIMA0_DAT renamed /REF_SLIMA0_DAT
- net /REF_SLIMA1_CLK renamed /REF_SLIMA1_CLK
- net /REF_SLIMA1_DAT renamed /REF_SLIMA1_DAT
- net /REF_SLIMA2_CLK renamed /REF_SLIMA2_CLK
- net /REF_SLIMA2_DAT renamed /REF_SLIMA2_DAT
- net /REF_SLIMA3_CLK renamed /REF_SLIMA3_CLK
- net /REF_SLIMA3_DAT renamed /REF_SLIMA3_DAT
- net /REF_SLIMB0_CLK renamed /REF_SLIMB0_CLK
- net /REF_SLIMB0_DAT renamed /REF_SLIMB0_DAT
- net /REF_SLIMB1_CLK renamed /REF_SLIMB1_CLK
- net /REF_SLIMB1_DAT renamed /REF_SLIMB1_DAT
- net /REF_SLIMB2_CLK renamed /REF_SLIMB2_CLK
- net /REF_SLIMB2_DAT renamed /REF_SLIMB2_DAT
- net /REF_SLIMB3_CLK renamed /REF_SLIMB3_CLK
- net /REF_SLIMB3_DAT renamed /REF_SLIMB3_DAT
- net /REF_SMB_A_A0 renamed /REF_SMB_A_A0
- net /REF_SMB_A_A1 renamed /REF_SMB_A_A1
- net /REF_SMB_A_A2 renamed /REF_SMB_A_A2
- net /REF_SMB_A_SCL renamed /REF_SMB_A_SCL
- net /REF_SMB_A_SDA renamed /REF_SMB_A_SDA
- net /REF_SRNS_REFCLKN renamed /REF_SRNS_REFCLKN
- net /REF_SRNS_REFCLKP renamed /REF_SRNS_REFCLKP
- net /TB5_CC1 renamed /TB5_CC1
- net /TB5_CC2 renamed /TB5_CC2
- net /TB5_RX1_N renamed /TB5_RX1_N
- net /TB5_RX1_P renamed /TB5_RX1_P
- net /TB5_RX2_N renamed /TB5_RX2_N
- net /TB5_RX2_P renamed /TB5_RX2_P
- net /TB5_SBU1 renamed /TB5_SBU1
- net /TB5_SBU2 renamed /TB5_SBU2
- net /TB5_TX1_N renamed /TB5_TX1_N
- net /TB5_TX1_P renamed /TB5_TX1_P
- net /TB5_TX2_N renamed /TB5_TX2_N
- net /TB5_TX2_P renamed /TB5_TX2_P
- net /TB5_USB2_DN renamed /TB5_USB2_DN
- net /TB5_USB2_DP renamed /TB5_USB2_DP
- net /TB5_VBUS renamed /TB5_VBUS
- net /VBANK_A renamed /VBANK_A
- net /VBANK_B renamed /VBANK_B
- net /VIN_A renamed /VIN_A
- net /VIN_B renamed /VIN_B
- J501 pad 50: /M1_PERST -> /M1_PERST
- J502 pad 50: /M2_PERST -> /M2_PERST
- J503 pad 50: /M3_PERST -> /M3_PERST
- J504 pad 50: /M4_PERST -> /M4_PERST
Routing:
- net /GND: track 0.00 -> 19.8 mm, vias 10 -> 18
- net /M2_PERST: track 0.00 -> 5.90 mm, vias 0 -> 2
- net /M1_PERST: track 0.00 -> 5.90 mm, vias 0 -> 2
- net /M4_PERST: track 0.00 -> 3.28 mm, vias 0 -> 2
- net /M3_PERST: track 0.00 -> 3.28 mm, vias 0 -> 2
