File: outputs/PCIe_E1S_96x45_USB12mm_RevW/Main_12E1S/Connectivity_55.kicad_sch (KiCad schematic)
At the start: 3 parts, among them Y501 25MHz / 20pF / 30ppm / ESR <=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, Y701 38.4MHz crystal / load and ES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, Y702 32.768kHz crystal / load and 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

Commit message: Reaudit retained E1S source and improve local converter current paths
Parts:
- added C9040: 100nF 6.3V X5R / U605 local bypass, Local:C_0201_DenseCourtyard_1p0x0p4, symbol Local:PART_C9040
- added R9040: 10k 1% / reset fail-low, Local:R_0201_DenseCourtyard_1p0x0p4, symbol Local:PART_R9040
Connections:
- net /GND: now also C9040.2, R9040.2
- new net /P3V3_AUX: C9040.1
- new net /TBT_PCIE_PERST_3V3_N: R9040.1
Other:
- note added: "U605 uses 3.3V AUX and U511 CPU PERST level translation with R9040 10k pulldown. Brownout/rail sequencing remain unqualified."
Changed lines of the file:
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@@
 (global_label "/CPU_RTCX1" (shape passive) (at 345.44 73.66 180) (effects (font (size 0.8 0.8)) (justify right)))
 (global_label "/CPU_RTCX2" (shape passive) (at 375.92 73.66 0) (effects (font (size 0.8 0.8)) (justify left)))
+(symbol (lib_id "Local:PART_C9040") (at 218.44 201.93 0) (unit 1) (in_bom yes) (on_board yes) (dnp no)
+(property "Reference" "C9040" (at 218.44 193.12 0) (effects (font (size 0.8 0.8))))
+(property "Value" "100nF 6.3V X5R / U605 local bypass" (at 218.44 190.12 0) (effects (font (size 0.8 0.8))))
+(property "Footprint" "Local:C_0201_DenseCourtyard_1p0x0p4" (at 218.44 201.93 0) (effects (font (size 0.8 0.8))))
+(pin "1") (pin "2")
+(instances (project "Main_12E1S" (path "/c33a6c5d-1a9e-4453-a37d-d3058a6ae0e3/6dd23699-f731-4167-b462-844d556d5ee1" (reference "C9040") (unit 1)))))
+(global_label "/P3V3_AUX" (shape passive) (at 203.2 201.93 180) (effects (font (size .8 .8)) (justify right)))
+(global_label "/GND" (shape passive) (at 233.68 201.93 0) (effects (font (size .8 .8)) (justify left)))
+(text "U605 uses 3.3V AUX and U511 CPU PERST level translation with R9040 10k pulldown. Brownout/rail sequencing remain unqualified." (at 20.32 238.76 0) (effects (font (size 1.27 1.27)) (justify left)))
+(symbol (lib_id "Local:PART_R9040") (at 504.19 201.93 0) (unit 1) (in_bom yes) (on_board yes) (dnp no) (property "Reference" "R9040" (at 504.19 193.12 0) (effects (font (size 1 1)))) (property "Value" "10k 1% / reset fail-low" (at 504.19 190.12 0) (effects (font (size 1 1)))) (property "Footprint" "Local:R_0201_DenseCourtyard_1p0x0p4" (at 504.19 201.93 0) (effects (font (size 1 1)) (hide yes))) (pin "1") (pin "2") (instances (project "Main_12E1S" (path "/c33a6c5d-1a9e-4453-a37d-d3058a6ae0e3/6dd23699-f731-4167-b462-844d556d5ee1" (reference "R9040") (unit 1)))))
+(global_label "/TBT_PCIE_PERST_3V3_N" (shape passive) (at 488.95 201.93 180) (effects (font (size .8 .8)) (justify right)))
+(global_label "/GND" (shape passive) (at 519.43 201.93 0) (effects (font (size .8 .8)) (justify left)))
 )
