File: outputs/PCIe_E1S_96x45_USB12mm_RevW/Main_12E1S/Main_12E1S.kicad_pcb (KiCad board)
At the start: 32 copper layers, 96 x 45 mm, 583 parts, among them J1 HSEC6-028-01-S-DV-WT-TR, J10 HSEC6-028-01-S-DV-WT-TR, J101 12V INPUT A / 20A budget / so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, J102 12V INPUT B / 20A budget / so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, J11 HSEC6-028-01-S-DV-WT-TR, J12 HSEC6-028-01-S-DV-WT-TR, J2 HSEC6-028-01-S-DV-WT-TR, J3 HSEC6-028-01-S-DV-WT-TR, J4 HSEC6-028-01-S-DV-WT-TR, J401 CUSTOM POWER USB-C / ISOLATED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, J402 THUNDERBOLT 3 HOST / VERTICAL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, J5 HSEC6-028-01-S-DV-WT-TR, J6 HSEC6-028-01-S-DV-WT-TR, J7 HSEC6-028-01-S-DV-WT-TR, J8 HSEC6-028-01-S-DV-WT-TR, J9 HSEC6-028-01-S-DV-WT-TR, U1 PEX90064 / FAKE 64-lane 33x33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, U11 TPS259470ARPWR, U12 TPS259470ARPWR, U13 TPS259470ARPWR, U14 TPS259470ARPWR, U15 TPS259470ARPWR, U16 TPS259470ARPWR, U17 TPS259470ARPWR, U18 TPS259470ARPWR, U19 TPS259470ARPWR, U20 TPS259470ARPWR, U21 TPS259470ARPWR, U22 TPS259470ARPWR, U30 TPS259470ARPWR, U31 TPS62132RGTR, U501 DSL6540 / Alpine Ridge DP / T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, U502 Intel Core Ultra 9 288V / 32G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, U503 TPS65982 / Type-C DFP / 5V3A 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, U504 W25Q80DVSNJG / 3.3V 8Mbit NVM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, U505 W25Q80DVSNJG / 3.3V 8Mbit NVM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, U506 TPS62133RGTR / 12V to 5V 3A U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, U510 TPS3808G33DBVR / AR reset del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, U511 SN74AXC1T45DCKR / PERST 1.8V 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, U512 SN74AXC1T45DCKR / HPDA 3.3V t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, U601 9ZXL0851EKILFT / CPU common c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, U602 9ZXL0851EKILFT / CPU common c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, U603 9FGV0241AKLF / DNP ALTERNATE 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, U604 9DML0451AKILF / DNP ALTERNATE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, U605 TPS3808G09DBVR / SUPPORT NETW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, U606 W25Q32JWSSIQ_C2980995 / SUPPO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, U607 TCA9548ARGER / SUPPORT NETWOR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, U701 W25Q256JWPIQ / 1.8V 32MiB BIOS, U702 TPS7A0215PDBVR / RTC 1.5V, U901 TPS548D22RVFR / 0.9004V 40A r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, U902 TPSM63610RDFR / 1.8V 8A, Y501 25MHz / 20pF / 30ppm / ESR <=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, Y701 38.4MHz crystal / load and ES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, Y702 32.768kHz crystal / load and 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

Commit message: Rebuild E1S reset routing and remove conflicting PLTRST pull-up
Parts:
- moved U605 50.0 mm to (34.0, 41.0), turned to 180 degrees
- moved R9040 50.0 mm to (36.5, 42.0), turned to 0 degrees
- moved C9040 45.0 mm to (31.4, 40.0), turned to 180 degrees
- moved R724 42.4 mm to (36.6, 40.2), turned to -90 degrees
- moved C741 22.1 mm to (31.0, 42.0), turned to 180 degrees
Routing:
- net /CPU_PERST_1V8_N: track 0.00 -> 47.4 mm, vias 0 -> 3
- net /TBT_PCIE_PERST_3V3_N: track 25.6 -> 71.2 mm, vias 2 -> 3
- net /PEX_SYS_RESET_N: track 0.00 -> 4.55 mm
- net /GND: track 24.3 -> 27.6 mm, vias 2080 -> 2081
- net /PEX_RESET_CT: track 0.00 -> 1.22 mm
- net /P3V3_AUX: track 4.80 -> 5.51 mm
- net /PEX_0V9: track 1.70 -> 2.40 mm
